Commit message: Add STEP-based robot visuals and walking stair demonstration

File: src/biped_description/urdf/base.xacro (robot description, xacro)
@@ -30,11 +30,5 @@
   <xacro:macro name="base" params="with_payload:=true">
     <link name="base_link">
-      <visual>
-        <origin xyz="0 0 0"/>
-        <geometry>
-          <box size="${pelvis_w} ${pelvis_d} ${pelvis_h}"/>
-        </geometry>
-        <material name="dark_grey"/>
-      </visual>
+      <xacro:cad_visual link="base_link"/>
       <collision>
         <origin xyz="0 0 0"/>
@@ -51,36 +45,5 @@
     </joint>
     <link name="platform_link">
-      <!-- Torso visual: white chest shell + teal chest panel + dark
-           shoulder bar, instead of the bare shelf slab. Visual-only;
-           the physics collision stays the original shelf so masses
-           and inertia are untouched. -->
-      <visual>
-        <origin xyz="0 0 ${0.055}"/>
-        <geometry>
-          <box size="0.17 0.17 0.14"/>
-        </geometry>
-        <material name="silver"/>
-      </visual>
-      <visual>
-        <origin xyz="0.088 0 0.06"/>
-        <geometry>
-          <box size="0.005 0.11 0.08"/>
-        </geometry>
-        <material name="accent_teal"/>
-      </visual>
-      <visual>
-        <origin xyz="0 0 ${0.135}"/>
-        <geometry>
-          <box size="0.24 0.09 0.045"/>
-        </geometry>
-        <material name="actuator_dark"/>
-      </visual>
-      <visual>
-        <origin xyz="0 0 0"/>
-        <geometry>
-          <box size="${plat_w} ${plat_d} ${plat_t}"/>
-        </geometry>
-        <material name="silver"/>
-      </visual>
+      <xacro:cad_visual link="platform_link"/>
       <collision>
         <origin xyz="0 0 0"/>
@@ -98,20 +61,5 @@
       </joint>
       <link name="payload_link">
-        <!-- Head module: white head shell + glowing cyan visor strip
-             on the front face. Visual-only; collision/inertia unchanged. -->
-        <visual>
-          <origin xyz="0 0 0"/>
-          <geometry>
-            <box size="0.10 0.10 0.08"/>
-          </geometry>
-          <material name="silver"/>
-        </visual>
-        <visual>
-          <origin xyz="0.0505 0 0.01"/>
-          <geometry>
-            <box size="0.002 0.085 0.028"/>
-          </geometry>
-          <material name="eye_cyan"/>
-        </visual>
+        <!-- No payload object appears in Robot.STEP. Its physics is retained. -->
         <collision>
           <origin xyz="0 0 0"/>

File: src/biped_description/urdf/biped.urdf.xacro (robot description, xacro)
@@ -9,17 +9,6 @@
   <xacro:arg name="with_payload" default="true"/>
   <xacro:property name="with_payload" value="$(arg with_payload)"/>
-  <!-- Shared materials -->
-  <material name="dark_grey"><color rgba="0.35 0.35 0.38 1.0"/></material>
-  <!-- 2026-09-21 visual redesign: white shell + teal accents (the old
-       0.75 grey read as raw lumber in screenshots). 'silver' kept as
-       the name because leg/platform visuals reference it. -->
-  <material name="silver"><color rgba="0.91 0.91 0.93 1.0"/></material>
-  <material name="accent_teal"><color rgba="0.05 0.60 0.62 1.0"/></material>
-  <material name="eye_cyan"><color rgba="0.30 0.95 1.00 1.0"/></material>
-  <material name="black"><color rgba="0.08 0.08 0.08 1.0"/></material>
-  <material name="payload_black"><color rgba="0.10 0.10 0.10 1.0"/></material>
-  <material name="torso_orange"><color rgba="0.85 0.35 0.05 1.0"/></material>
-  <material name="eye_white"><color rgba="0.95 0.95 0.95 1.0"/></material>
-  <material name="actuator_dark"><color rgba="0.10 0.10 0.12 1.0"/></material>
+  <!-- Appearance from Robot.STEP; all simulation parameters stay original. -->
+  <xacro:include filename="cad_visuals.xacro"/>
   <xacro:include filename="inertia.xacro"/>
   <xacro:include filename="base.xacro"/>

File: src/biped_description/urdf/leg.xacro (robot description, xacro)
@@ -57,9 +57,5 @@
     </joint>
     <link name="${prefix}_hip_pitch_link">
-      <visual>
-        <origin xyz="0 0 0"/>
-        <geometry><cylinder radius="0.045" length="0.07"/></geometry>
-        <material name="actuator_dark"/>
-      </visual>
+      <xacro:cad_visual link="${prefix}_hip_pitch_link"/>
       <collision>
         <origin xyz="0 0 0"/>
@@ -79,16 +75,5 @@
     <!-- Thigh: from hip down to knee -->
     <link name="${prefix}_thigh">
-      <visual>
-        <origin xyz="0 0 ${-thigh_len/2}"/>
-        <geometry><box size="${thigh_w} ${thigh_d} ${thigh_len}"/></geometry>
-        <material name="silver"/>
-      </visual>
-      <!-- Knee actuator disc: visual-only (matches Robot.png); no collision
-           element so Gazebo contacts stay clean between adjacent links. -->
-      <visual>
-        <origin xyz="0 0 ${-thigh_len}"/>
-        <geometry><cylinder radius="0.05" length="0.055"/></geometry>
-        <material name="actuator_dark"/>
-      </visual>
+      <xacro:cad_visual link="${prefix}_thigh"/>
       <collision>
         <origin xyz="0 0 ${-thigh_len/2}"/>
@@ -109,9 +94,5 @@
     <!-- Shin: from knee down to ankle -->
     <link name="${prefix}_shin">
-      <visual>
-        <origin xyz="0 0 ${-shin_len/2}"/>
-        <geometry><box size="${shin_w} ${shin_d} ${shin_len}"/></geometry>
-        <material name="silver"/>
-      </visual>
+      <xacro:cad_visual link="${prefix}_shin"/>
       <collision>
         <origin xyz="0 0 ${-shin_len/2}"/>
@@ -131,18 +112,5 @@
     </joint>
     <link name="${prefix}_ankle_roll_link">
-      <visual>
-        <origin xyz="0 0 0"/>
-        <geometry><cylinder radius="0.04" length="0.05"/></geometry>
-        <material name="actuator_dark"/>
-      </visual>
-      <!-- Ankle-to-foot connector: the shin ends AT the ankle axis and
-           the foot box top is 12 cm lower - without this the foot
-           looked detached, floating in air. Visual-only (no collision):
-           the sole must stay the only foot contact for the M8 sensors. -->
-      <visual>
-        <origin xyz="0 0 ${-0.06}"/>
-        <geometry><box size="0.03 0.04 0.12"/></geometry>
-        <material name="actuator_dark"/>
-      </visual>
+      <!-- The CAD ankle assembly is included in the foot visual. -->
       <collision>
         <origin xyz="0 0 0"/>
@@ -168,9 +136,5 @@
          silently matches nothing - found the hard way in M8 testing. -->
     <link name="${prefix}_foot">
-      <visual>
-        <origin xyz="0.02 0 ${-ankle_h + foot_h/2}"/>
-        <geometry><box size="${foot_len} ${foot_w} ${foot_h}"/></geometry>
-        <material name="black"/>
-      </visual>
+      <xacro:cad_visual link="${prefix}_foot"/>
       <collision>
         <origin xyz="0.02 0 ${-ankle_h + foot_h/2}"/>
